Commit message: Robot in Gazebo
Added an extra package to configure the gazebo world. Will be removed in the future

File: robots/src/upper_14_back/urdf/lita.urdf (robot description, URDF)
Before this commit: robot lita_converted, 16 links, 15 joints
Links:
- link l_elbow_link: geometry collision mesh filename=package://upper_14/meshes/l_elbow_link.STL; visual mesh filename=package://upper_14/meshes/l_elbow_link.STL
- link l_shoulder_pitch_link: geometry collision mesh filename=package://upper_14/meshes/l_shoulder_pitch_link.STL; visual mesh filename=package://upper_14/meshes/l_shoulder_pitch_link.STL
- link l_shoulder_roll_link: geometry collision mesh filename=package://upper_14/meshes/l_shoulder_roll_link.STL; visual mesh filename=package://upper_14/meshes/l_shoulder_roll_link.STL
- link l_shoulder_yaw_link: geometry collision mesh filename=package://upper_14/meshes/l_shoulder_yaw_link.STL; visual mesh filename=package://upper_14/meshes/l_shoulder_yaw_link.STL
- link l_wrist_pitch_link: geometry collision mesh filename=package://upper_14/meshes/l_wrist_pitch_link.STL; visual mesh filename=package://upper_14/meshes/l_wrist_pitch_link.STL
- link l_wrist_roll_link: geometry collision mesh filename=package://upper_14/meshes/l_wrist_roll_link.STL; visual mesh filename=package://upper_14/meshes/l_wrist_roll_link.STL
- link l_wrist_yaw_link: geometry collision mesh filename=package://upper_14/meshes/l_wrist_yaw_link.STL; visual mesh filename=package://upper_14/meshes/l_wrist_yaw_link.STL
- link r_elbow_link: geometry collision mesh filename=package://upper_14/meshes/r_elbow_link.STL; visual mesh filename=package://upper_14/meshes/r_elbow_link.STL
- link r_shoulder_pitch_link: geometry collision mesh filename=package://upper_14/meshes/r_shoulder_pitch_link.STL; visual mesh filename=package://upper_14/meshes/r_shoulder_pitch_link.STL
- link r_shoulder_roll_link: geometry collision mesh filename=package://upper_14/meshes/r_shoulder_roll_link.STL; visual mesh filename=package://upper_14/meshes/r_shoulder_roll_link.STL
- link r_shoulder_yaw_link: geometry collision mesh filename=package://upper_14/meshes/r_shoulder_yaw_link.STL; visual mesh filename=package://upper_14/meshes/r_shoulder_yaw_link.STL
- link r_wrist_pitch_link: geometry collision mesh filename=package://upper_14/meshes/r_wrist_pitch_link.STL; visual mesh filename=package://upper_14/meshes/r_wrist_pitch_link.STL
- link r_wrist_roll_link: geometry collision mesh filename=package://upper_14/meshes/r_wrist_roll_link.STL; visual mesh filename=package://upper_14/meshes/r_wrist_roll_link.STL
- link r_wrist_yaw_link: geometry collision mesh filename=package://upper_14/meshes/r_wrist_yaw_link.STL; visual mesh filename=package://upper_14/meshes/r_wrist_yaw_link.STL
- link upper_body_link: geometry collision mesh filename=package://upper_14/meshes/upper_body_link.STL; visual mesh filename=package://upper_14/meshes/upper_body_link.STL

File: robots/src/upper_14_back/urdf/lita.xacro (robot description, xacro)
@@ -1,4 +1,4 @@
 <?xml version="1.0"?>
-<robot name="lita_converted" xmlns:xacro="http://www.ros.org/wiki/xacro">
+<robot name="upper_14" xmlns:xacro="http://www.ros.org/wiki/xacro">
   <!--fix the upper_body_link-->
   <link name="world"/>
@@ -20,5 +20,5 @@
       <origin xyz="0 0 0" rpy="0 0 0" />
       <geometry>
-        <mesh filename="package://lita_converted/meshes/upper_body_link.STL" />
+        <mesh filename="package://upper_14/meshes/upper_body_link.STL" />
       </geometry>
       <material name="">
@@ -29,5 +29,5 @@
       <origin xyz="0 0 0" rpy="0 0 0" />
       <geometry>
-        <mesh filename="package://lita_converted/meshes/upper_body_link.STL" />
+        <mesh filename="package://upper_14/meshes/upper_body_link.STL" />
       </geometry>
     </collision>
@@ -56,5 +56,5 @@
       <geometry>
         <mesh
-          filename="package://lita_converted/meshes/l_shoulder_roll_link.STL" />
+          filename="package://upper_14/meshes/l_shoulder_roll_link.STL" />
       </geometry>
       <material name="">
@@ -66,5 +66,5 @@
       <geometry>
         <mesh
-          filename="package://lita_converted/meshes/l_shoulder_roll_link.STL" />
+          filename="package://upper_14/meshes/l_shoulder_roll_link.STL" />
       </geometry>
     </collision>
@@ -92,19 +92,19 @@
       <geometry>
         <mesh
-          filename="package://lita_converted/meshes/l_shoulder_pitch_link.STL" />
-      </geometry>
-      <material
-        name="">
-        <color
-          rgba="0.68627 0.65882 0.63922 1" />
-      </material>
-    </visual>
-    <collision>
-      <origin
-        xyz="0 0 0"
-        rpy="0 0 0" />
-      <geometry>
-        <mesh
-          filename="package://lita_converted/meshes/l_shoulder_pitch_link.STL" />
+          filename="package://upper_14/meshes/l_shoulder_pitch_link.STL" />
+      </geometry>
+      <material
+        name="">
+        <color
+          rgba="0.68627 0.65882 0.63922 1" />
+      </material>
+    </visual>
+    <collision>
+      <origin
+        xyz="0 0 0"
+        rpy="0 0 0" />
+      <geometry>
+        <mesh
+          filename="package://upper_14/meshes/l_shoulder_pitch_link.STL" />
       </geometry>
     </collision>
@@ -160,19 +160,19 @@
       <geometry>
         <mesh
-          filename="package://lita_converted/meshes/l_shoulder_yaw_link.STL" />
-      </geometry>
-      <material
-        name="">
-        <color
-          rgba="0.68627 0.65882 0.63922 1" />
-      </material>
-    </visual>
-    <collision>
-      <origin
-        xyz="0 0 0"
-        rpy="0 0 0" />
-      <geometry>
-        <mesh
-          filename="package://lita_converted/meshes/l_shoulder_yaw_link.STL" />
+          filename="package://upper_14/meshes/l_shoulder_yaw_link.STL" />
+      </geometry>
+      <material
+        name="">
+        <color
+          rgba="0.68627 0.65882 0.63922 1" />
+      </material>
+    </visual>
+    <collision>
+      <origin
+        xyz="0 0 0"
+        rpy="0 0 0" />
+      <geometry>
+        <mesh
+          filename="package://upper_14/meshes/l_shoulder_yaw_link.STL" />
       </geometry>
     </collision>
@@ -228,19 +228,19 @@
       <geometry>
         <mesh
-          filename="package://lita_converted/meshes/l_elbow_link.STL" />
-      </geometry>
-      <material
-        name="">
-        <color
-          rgba="0.68627 0.65882 0.63922 1" />
-      </material>
-    </visual>
-    <collision>
-      <origin
-        xyz="0 0 0"
-        rpy="0 0 0" />
-      <geometry>
-        <mesh
-          filename="package://lita_converted/meshes/l_elbow_link.STL" />
+          filename="package://upper_14/meshes/l_elbow_link.STL" />
+      </geometry>
+      <material
+        name="">
+        <color
+          rgba="0.68627 0.65882 0.63922 1" />
+      </material>
+    </visual>
+    <collision>
+      <origin
+        xyz="0 0 0"
+        rpy="0 0 0" />
+      <geometry>
+        <mesh
+          filename="package://upper_14/meshes/l_elbow_link.STL" />
       </geometry>
     </collision>
@@ -296,19 +296,19 @@
       <geometry>
         <mesh
-          filename="package://lita_converted/meshes/l_wrist_roll_link.STL" />
-      </geometry>
-      <material
-        name="">
-        <color
-          rgba="0.68627 0.65882 0.63922 1" />
-      </material>
-    </visual>
-    <collision>
-      <origin
-        xyz="0 0 0"
-        rpy="0 0 0" />
-      <geometry>
-        <mesh
-          filename="package://lita_converted/meshes/l_wrist_roll_link.STL" />
+          filename="package://upper_14/meshes/l_wrist_roll_link.STL" />
+      </geometry>
+      <material
+        name="">
+        <color
+          rgba="0.68627 0.65882 0.63922 1" />
+      </material>
+    </visual>
+    <collision>
+      <origin
+        xyz="0 0 0"
+        rpy="0 0 0" />
+      <geometry>
+        <mesh
+          filename="package://upper_14/meshes/l_wrist_roll_link.STL" />
       </geometry>
     </collision>
@@ -359,19 +359,19 @@
       <geometry>
         <mesh
-          filename="package://lita_converted/meshes/l_wrist_pitch_link.STL" />
-      </geometry>
-      <material
-        name="">
-        <color
-          rgba="0.68627 0.65882 0.63922 1" />
-      </material>
-    </visual>
-    <collision>
-      <origin
-        xyz="0 0 0"
-        rpy="0 0 0" />
-      <geometry>
-        <mesh
-          filename="package://lita_converted/meshes/l_wrist_pitch_link.STL" />
+          filename="package://upper_14/meshes/l_wrist_pitch_link.STL" />
+      </geometry>
+      <material
+        name="">
+        <color
+          rgba="0.68627 0.65882 0.63922 1" />
+      </material>
+    </visual>
+    <collision>
+      <origin
+        xyz="0 0 0"
+        rpy="0 0 0" />
+      <geometry>
+        <mesh
+          filename="package://upper_14/meshes/l_wrist_pitch_link.STL" />
       </geometry>
     </collision>
@@ -427,19 +427,19 @@
       <geometry>
         <mesh
-          filename="package://lita_converted/meshes/l_wrist_yaw_link.STL" />
-      </geometry>
-      <material
-        name="">
-        <color
-          rgba="0.68627 0.65882 0.63922 1" />
-      </material>
-    </visual>
-    <collision>
-      <origin
-        xyz="0 0 0"
-        rpy="0 0 0" />
-      <geometry>
-        <mesh
-          filename="package://lita_converted/meshes/l_wrist_yaw_link.STL" />
+          filename="package://upper_14/meshes/l_wrist_yaw_link.STL" />
+      </geometry>
+      <material
+        name="">
+        <color
+          rgba="0.68627 0.65882 0.63922 1" />
+      </material>
+    </visual>
+    <collision>
+      <origin
+        xyz="0 0 0"
+        rpy="0 0 0" />
+      <geometry>
+        <mesh
+          filename="package://upper_14/meshes/l_wrist_yaw_link.STL" />
       </geometry>
     </collision>
@@ -495,19 +495,19 @@
       <geometry>
         <mesh
-          filename="package://lita_converted/meshes/r_shoulder_roll_link.STL" />
-      </geometry>
-      <material
-        name="">
-        <color
-          rgba="0.68627 0.65882 0.63922 1" />
-      </material>
-    </visual>
-    <collision>
-      <origin
-        xyz="0 0 0"
-        rpy="0 0 0" />
-      <geometry>
-        <mesh
-          filename="package://lita_converted/meshes/r_shoulder_roll_link.STL" />
+          filename="package://upper_14/meshes/r_shoulder_roll_link.STL" />
+      </geometry>
+      <material
+        name="">
+        <color
+          rgba="0.68627 0.65882 0.63922 1" />
+      </material>
+    </visual>
+    <collision>
+      <origin
+        xyz="0 0 0"
+        rpy="0 0 0" />
+      <geometry>
+        <mesh
+          filename="package://upper_14/meshes/r_shoulder_roll_link.STL" />
       </geometry>
     </collision>
@@ -558,19 +558,19 @@
       <geometry>
         <mesh
-          filename="package://lita_converted/meshes/r_shoulder_pitch_link.STL" />
-      </geometry>
-      <material
-        name="">
-        <color
-          rgba="0.68627 0.65882 0.63922 1" />
-      </material>
-    </visual>
-    <collision>
-      <origin
-        xyz="0 0 0"
-        rpy="0 0 0" />
-      <geometry>
-        <mesh
-          filename="package://lita_converted/meshes/r_shoulder_pitch_link.STL" />
+          filename="package://upper_14/meshes/r_shoulder_pitch_link.STL" />
+      </geometry>
+      <material
+        name="">
+        <color
+          rgba="0.68627 0.65882 0.63922 1" />
+      </material>
+    </visual>
+    <collision>
+      <origin
+        xyz="0 0 0"
+        rpy="0 0 0" />
+      <geometry>
+        <mesh
+          filename="package://upper_14/meshes/r_shoulder_pitch_link.STL" />
       </geometry>
     </collision>
@@ -626,19 +626,19 @@
       <geometry>
         <mesh
-          filename="package://lita_converted/meshes/r_shoulder_yaw_link.STL" />
-      </geometry>
-      <material
-        name="">
-        <color
-          rgba="0.68627 0.65882 0.63922 1" />
-      </material>
-    </visual>
-    <collision>
-      <origin
-        xyz="0 0 0"
-        rpy="0 0 0" />
-      <geometry>
-        <mesh
-          filename="package://lita_converted/meshes/r_shoulder_yaw_link.STL" />
+          filename="package://upper_14/meshes/r_shoulder_yaw_link.STL" />
+      </geometry>
+      <material
+        name="">
+        <color
+          rgba="0.68627 0.65882 0.63922 1" />
+      </material>
+    </visual>
+    <collision>
+      <origin
+        xyz="0 0 0"
+        rpy="0 0 0" />
+      <geometry>
+        <mesh
+          filename="package://upper_14/meshes/r_shoulder_yaw_link.STL" />
       </geometry>
     </collision>
@@ -693,19 +693,19 @@
       <geometry>
         <mesh
-          filename="package://lita_converted/meshes/r_elbow_link.STL" />
-      </geometry>
-      <material
-        name="">
-        <color
-          rgba="0.68627 0.65882 0.63922 1" />
-      </material>
-    </visual>
-    <collision>
-      <origin
-        xyz="0 0 0"
-        rpy="0 0 0" />
-      <geometry>
-        <mesh
-          filename="package://lita_converted/meshes/r_elbow_link.STL" />
+          filename="package://upper_14/meshes/r_elbow_link.STL" />
+      </geometry>
+      <material
+        name="">
+        <color
+          rgba="0.68627 0.65882 0.63922 1" />
+      </material>
+    </visual>
+    <collision>
+      <origin
+        xyz="0 0 0"
+        rpy="0 0 0" />
+      <geometry>
+        <mesh
+          filename="package://upper_14/meshes/r_elbow_link.STL" />
       </geometry>
     </collision>
@@ -761,19 +761,19 @@
       <geometry>
         <mesh
-          filename="package://lita_converted/meshes/r_wrist_roll_link.STL" />
-      </geometry>
-      <material
-        name="">
-        <color
-          rgba="0.68627 0.65882 0.63922 1" />
-      </material>
-    </visual>
-    <collision>
-      <origin
-        xyz="0 0 0"
-        rpy="0 0 0" />
-      <geometry>
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