Commit message: links ready in gazebo
links correctly configured

File: robots/src/upper_14/urdf/lita.xacro (robot description, xacro)
@@ -45,16 +45,12 @@
       <mass value="0.63417" />
       <inertia
-        ixx="0.000315"
-        ixy="0"
-        ixz="-5.2E-05"
-        iyy="0.000373"
-        iyz="0"
+        ixx="0.000315" ixy="0" ixz="-5.2E-05"
+        iyy="0.000373" iyz="0"
         izz="0.000525" />
     </inertial>
     <visual>
-      <origin xyz="0.125 0 0.26" rpy="0 -1.5708 0" />
-      <geometry>
-        <mesh
-          filename="package://upper_14/meshes/l_shoulder_roll_link.STL" />
+      <origin xyz="0 0 0" rpy="0 0 0" />
+      <geometry>
+        <mesh filename="package://upper_14/meshes/l_shoulder_roll_link.STL" />
       </geometry>
       <material name="">
@@ -63,277 +59,151 @@
     </visual>
     <collision>
-      <origin xyz="0.125 0 0.26" rpy="0 -1.5708 0" />
-      <geometry>
-        <mesh
-          filename="package://upper_14/meshes/l_shoulder_roll_link.STL" />
-      </geometry>
-    </collision>
-  </link>
-  <link
-    name="l_shoulder_pitch_link">
-    <inertial>
-      <origin
-        xyz="0.0032993 5.9585E-10 -0.00098089"
-        rpy="0 0 0" />
-      <mass
-        value="1.0724" />
-      <inertia
-        ixx="0.000841"
-        ixy="0"
-        ixz="-5.4E-05"
-        iyy="0.000973"
-        iyz="0"
+      <origin xyz="0 0 0" rpy="0 0 0" />
+      <geometry>
+        <mesh filename="package://upper_14/meshes/l_shoulder_roll_link.STL" />
+      </geometry>
+    </collision>
+  </link>
+  <link name="l_shoulder_pitch_link">
+    <inertial>
+      <origin xyz="0.0032993 5.9585E-10 -0.00098089" rpy="0 0 0" />
+      <mass value="1.0724" />
+      <inertia
+        ixx="0.000841" ixy="0" ixz="-5.4E-05"
+        iyy="0.000973" iyz="0"
         izz="0.000606" />
     </inertial>
     <visual>
-      <origin
-        xyz="0 0 0"
-        rpy="0 0 0" />
-      <geometry>
-        <mesh
-          filename="package://upper_14/meshes/l_shoulder_pitch_link.STL" />
-      </geometry>
-      <material
-        name="">
-        <color
-          rgba="0.68627 0.65882 0.63922 1" />
-      </material>
-    </visual>
-    <collision>
-      <origin
-        xyz="0 0 0"
-        rpy="0 0 0" />
-      <geometry>
-        <mesh
-          filename="package://upper_14/meshes/l_shoulder_pitch_link.STL" />
-      </geometry>
-    </collision>
-  </link>
-  <joint
-    name="l_shoulder_pitch"
-    type="revolute">
-    <origin
-      xyz="-0.0037133 0 -0.052049"
-      rpy="1.5708 1.5708 0" />
-    <parent
-      link="l_shoulder_roll_link" />
-    <child
-      link="l_shoulder_pitch_link" />
-    <axis
-      xyz="0 0 -1" />
-    <limit
-      lower="-0.6981"
-      upper="1.7104"
-      effort="50000"
-      velocity="500" />
-    <calibration
-      rising="1" />
-    <dynamics
-      damping="0.1"
-      friction="0.1" />
-    <safety_controller
-      soft_upper="1.7"
-      soft_lower="-0.69"
-      k_position="1"
-      k_velocity="1" />
-  </joint>
-  <link
-    name="l_shoulder_yaw_link">
-    <inertial>
-      <origin
-        xyz="0.065121 -0.0020967 1.7569E-07"
-        rpy="0 0 0" />
-      <mass
-        value="1.3826" />
-      <inertia
-        ixx="0.000398"
-        ixy="-0.000132"
-        ixz="0"
-        iyy="0.005026"
-        iyz="0"
+      <origin xyz="0 0 0" rpy="0 0 0" />
+      <geometry>
+        <mesh filename="package://upper_14/meshes/l_shoulder_pitch_link.STL" />
+      </geometry>
+      <material name="">
+        <color rgba="0.68627 0.65882 0.63922 1" />
+      </material>
+    </visual>
+    <collision>
+      <origin xyz="0 0 0" rpy="0 0 0" />
+      <geometry>
+        <mesh filename="package://upper_14/meshes/l_shoulder_pitch_link.STL" />
+      </geometry>
+    </collision>
+  </link>
+  <joint name="l_shoulder_pitch" type="revolute">
+    <origin xyz="-0.0037133 0 -0.052049" rpy="1.5708 1.5708 0" />
+    <parent link="l_shoulder_roll_link" />
+    <child link="l_shoulder_pitch_link" />
+    <axis xyz="0 0 -1" />
+    <limit lower="-0.6981" upper="1.7104" effort="50000" velocity="500" />
+    <calibration rising="1" />
+    <dynamics damping="0.7" friction="0.1" />
+    <safety_controller soft_upper="1.7" soft_lower="-0.69" k_position="1" k_velocity="1" />
+  </joint>
+  <link name="l_shoulder_yaw_link">
+    <inertial>
+      <origin xyz="0.065121 -0.0020967 1.7569E-07" rpy="0 0 0" />
+      <mass value="1.3826" />
+      <inertia
+        ixx="0.000398" ixy="-0.000132" ixz="0"
+        iyy="0.005026" iyz="0"
         izz="0.005143" />
     </inertial>
     <visual>
-      <origin
-        xyz="0 0 0"
-        rpy="0 0 0" />
-      <geometry>
-        <mesh
-          filename="package://upper_14/meshes/l_shoulder_yaw_link.STL" />
-      </geometry>
-      <material
-        name="">
-        <color
-          rgba="0.68627 0.65882 0.63922 1" />
-      </material>
-    </visual>
-    <collision>
-      <origin
-        xyz="0 0 0"
-        rpy="0 0 0" />
-      <geometry>
-        <mesh
-          filename="package://upper_14/meshes/l_shoulder_yaw_link.STL" />
-      </geometry>
-    </collision>
-  </link>
-  <joint
-    name="l_shoulder_yaw"
-    type="revolute">
-    <origin
-      xyz="0.055 0 0"
-      rpy="1.5708 -4.1633E-17 -2.6021E-18" />
-    <parent
-      link="l_shoulder_pitch_link" />
-    <child
-      link="l_shoulder_yaw_link" />
-    <axis
-      xyz="0 0 1" />
-    <limit
-      lower="-0.1396"
-      upper="1.6231"
-      effort="50000"
-      velocity="500" />
-    <calibration
-      rising="1" />
-    <dynamics
-      damping="0.1"
-      friction="0.1" />
-    <safety_controller
-      soft_upper="1.61"
-      soft_lower="-0.13"
-      k_position="1"
-      k_velocity="1" />
-  </joint>
-  <link
-    name="l_elbow_link">
-    <inertial>
-      <origin
-        xyz="0.088184 -0.0003499 -1.9687E-07"
-        rpy="0 0 0" />
-      <mass
-        value="0.81599" />
-      <inertia
-        ixx="0.000143"
-        ixy="1.5E-05"
-        ixz="0"
-        iyy="0.004114"
-        iyz="0"
+      <origin xyz="0 0 0" rpy="0 0 0" />
+      <geometry>
+        <mesh filename="package://upper_14/meshes/l_shoulder_yaw_link.STL" />
+      </geometry>
+      <material name="">
+        <color rgba="0.68627 0.65882 0.63922 1" />
+      </material>
+    </visual>
+    <collision>
+      <origin xyz="0 0 0" rpy="0 0 0" />
+      <geometry>
+        <mesh filename="package://upper_14/meshes/l_shoulder_yaw_link.STL" />
+      </geometry>
+    </collision>
+  </link>
+  <joint name="l_shoulder_yaw" type="revolute">
+    <origin xyz="0.055 0 0" rpy="1.5708 -4.1633E-17 -2.6021E-18" />
+    <parent link="l_shoulder_pitch_link" />
+    <child link="l_shoulder_yaw_link" />
+    <axis xyz="0 0 1" />
+    <limit lower="-0.1396" upper="1.6231" effort="50000" velocity="500" />
+    <calibration rising="1" />
+    <dynamics damping="0.7" friction="0.1" />
+    <safety_controller soft_upper="1.61" soft_lower="-0.13" k_position="1" k_velocity="1" />
+  </joint>
+  <link name="l_elbow_link">
+    <inertial>
+      <origin xyz="0.088184 -0.0003499 -1.9687E-07" rpy="0 0 0" />
+      <mass value="0.81599" />
+      <inertia
+        ixx="0.000143" ixy="1.5E-05" ixz="0"
+        iyy="0.004114" iyz="0"
         izz="0.004046" />
     </inertial>
     <visual>
-      <origin
-        xyz="0 0 0"
-        rpy="0 0 0" />
-      <geometry>
-        <mesh
-          filename="package://upper_14/meshes/l_elbow_link.STL" />
-      </geometry>
-      <material
-        name="">
-        <color
-          rgba="0.68627 0.65882 0.63922 1" />
-      </material>
-    </visual>
-    <collision>
-      <origin
-        xyz="0 0 0"
-        rpy="0 0 0" />
-      <geometry>
-        <mesh
-          filename="package://upper_14/meshes/l_elbow_link.STL" />
-      </geometry>
-    </collision>
-  </link>
-  <joint
-    name="l_elbow"
-    type="revolute">
-    <origin
-      xyz="0.1903 0 0"
-      rpy="-4.2858E-16 9.6277E-17 -4.1263E-32" />
-    <parent
-      link="l_shoulder_yaw_link" />
-    <child
-      link="l_elbow_link" />
-    <axis
-      xyz="0 0 1" />
-    <limit
-      lower="-0.7853"
-      upper="2.4085"
-      effort="50000"
-      velocity="500" />
-    <calibration
-      rising="1" />
-    <dynamics
-      damping="0.1"
-      friction="0.1" />
-    <safety_controller
-      soft_upper="2.4"
-      soft_lower="-0.78"
-      k_position="1"
-      k_velocity="1" />
-  </joint>
-  <link
-    name="l_wrist_roll_link">
-    <inertial>
-      <origin
-        xyz="-1.4822E-09 1.5222E-08 -0.0042713"
-        rpy="0 0 0" />
-      <mass
-        value="0.033212" />
-      <inertia
-        ixx="3E-06"
-        ixy="0"
-        ixz="0"
-        iyy="6E-06"
-        iyz="0"
+      <origin xyz="0 0 0" rpy="0 0 0" />
+      <geometry>
+        <mesh filename="package://upper_14/meshes/l_elbow_link.STL" />
+      </geometry>
+      <material
+        name="">
+        <color rgba="0.68627 0.65882 0.63922 1" />
+      </material>
+    </visual>
+    <collision>
+      <origin xyz="0 0 0" rpy="0 0 0" />
+      <geometry>
+        <mesh filename="package://upper_14/meshes/l_elbow_link.STL" />
+      </geometry>
+    </collision>
+  </link>
+  <joint name="l_elbow" type="revolute">
+    <origin xyz="0.1903 0 0" rpy="-4.2858E-16 9.6277E-17 -4.1263E-32" />
+    <parent link="l_shoulder_yaw_link" />
+    <child link="l_elbow_link" />
+    <axis xyz="0 0 1" />
+    <limit lower="-0.7853" upper="2.4085" effort="50000" velocity="500" />
+    <calibration rising="1" />
+    <dynamics damping="0.7" friction="0.1" />
+    <safety_controller soft_upper="2.4" soft_lower="-0.78" k_position="1" k_velocity="1" />
+  </joint>
+  <link name="l_wrist_roll_link">
+    <inertial>
+      <origin xyz="-1.4822E-09 1.5222E-08 -0.0042713" rpy="0 0 0" />
+      <mass value="0.033212" />
+      <inertia
+        ixx="3E-06" ixy="0" ixz="0"
+        iyy="6E-06" iyz="0"
         izz="8E-06" />
     </inertial>
     <visual>
-      <origin
-        xyz="0 0 0"
-        rpy="0 0 0" />
-      <geometry>
-        <mesh
-          filename="package://upper_14/meshes/l_wrist_roll_link.STL" />
-      </geometry>
-      <material
-        name="">
-        <color
-          rgba="0.68627 0.65882 0.63922 1" />
-      </material>
-    </visual>
-    <collision>
-      <origin
-        xyz="0 0 0"
-        rpy="0 0 0" />
-      <geometry>
-        <mesh
-          filename="package://upper_14/meshes/l_wrist_roll_link.STL" />
-      </geometry>
-    </collision>
-  </link>
-  <joint
-    name="l_wrist_roll"
-    type="continuous">
-    <origin
-      xyz="0.21 0 0"
-      rpy="3.1416 1.5708 0" />
-    <parent
-      link="l_elbow_link" />
-    <child
-      link="l_wrist_roll_link" />
-    <axis
-      xyz="0 0 -1" />
-    <limit
-      effort="50000"
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
Commit message: Robot Ready
The robot is current ready for the simulation. There's an issue that due to the lacking of  controller, the model will collapse to origin unless. The inertia matrix is changed to maintain stable, which can be restored from backup files.

File: robots/src/upper_14/urdf/lita.xacro (robot description, xacro)
@@ -1,3 +1,2 @@
-<?xml version="1.0"?>
 <robot name="upper_14" xmlns:xacro="http://www.ros.org/wiki/xacro">
   <!--fix the upper_body_link-->
@@ -37,6 +36,6 @@
     <parent link="upper_body_link" />
     <child link="l_shoulder_roll_link" />
-    <axis xyz="0 0 -1" />
-    <dynamics damping="0.7" />
+    <axis xyz="0 0 1" />
+    <dynamics damping="0.7" friction="0.2"/>
   </joint>
   <link name="l_shoulder_roll_link">
@@ -96,7 +95,5 @@
     <axis xyz="0 0 -1" />
     <limit lower="-0.6981" upper="1.7104" effort="50000" velocity="500" />
-    <calibration rising="1" />
-    <dynamics damping="0.7" friction="0.1" />
-    <safety_controller soft_upper="1.7" soft_lower="-0.69" k_position="1" k_velocity="1" />
+    <dynamics damping="0.7" friction="0.2"  />
   </joint>
   <link name="l_shoulder_yaw_link">
@@ -131,7 +128,5 @@
     <axis xyz="0 0 1" />
     <limit lower="-0.1396" upper="1.6231" effort="50000" velocity="500" />
-    <calibration rising="1" />
-    <dynamics damping="0.7" friction="0.1" />
-    <safety_controller soft_upper="1.61" soft_lower="-0.13" k_position="1" k_velocity="1" />
+    <dynamics damping="0.7" friction="0.2"  />
   </joint>
   <link name="l_elbow_link">
@@ -149,6 +144,5 @@
         <mesh filename="package://upper_14/meshes/l_elbow_link.STL" />
       </geometry>
-      <material
-        name="">
+      <material name="">
         <color rgba="0.68627 0.65882 0.63922 1" />
       </material>
@@ -167,7 +161,5 @@
     <axis xyz="0 0 1" />
     <limit lower="-0.7853" upper="2.4085" effort="50000" velocity="500" />
-    <calibration rising="1" />
-    <dynamics damping="0.7" friction="0.1" />
-    <safety_controller soft_upper="2.4" soft_lower="-0.78" k_position="1" k_velocity="1" />
+    <dynamics damping="0.7" friction="0.2"  />
   </joint>
   <link name="l_wrist_roll_link">
@@ -185,6 +177,5 @@
         <mesh filename="package://upper_14/meshes/l_wrist_roll_link.STL" />
       </geometry>
-      <material
-        name="">
+      <material name="">
         <color rgba="0.68627 0.65882 0.63922 1" />
       </material>
@@ -201,610 +192,450 @@
     <parent link="l_elbow_link" />
     <child link="l_wrist_roll_link" />
+    <axis xyz="0 0 1" />
+    <limit effort="50000" velocity="500" />
+    <dynamics damping="0.7" friction="0.2"  />
+  </joint>
+  <link name="l_wrist_pitch_link">
+    <inertial>
+      <origin xyz="0.0009785 -2.8101E-08 -1.4985E-08" rpy="0 0 0" />
+      <mass value="0.13385" />
+      <inertia
+        ixx="2.1E-03" ixy="0" ixz="0"
+        iyy="2.2E-03" iyz="0"
+        izz="2.2E-03" />
+    </inertial>
+    <visual>
+      <origin xyz="0 0 0" rpy="0 0 0" />
+      <geometry>
+        <mesh filename="package://upper_14/meshes/l_wrist_pitch_link.STL" />
+      </geometry>
+      <material name="">
+        <color rgba="0.68627 0.65882 0.63922 1" />
+      </material>
+    </visual>
+    <collision>
+      <origin xyz="0 0 0" rpy="0 0 0" />
+      <geometry>
+        <mesh filename="package://upper_14/meshes/l_wrist_pitch_link.STL" />
+      </geometry>
+    </collision>
+  </link>
+  <joint name="l_wrist_pitch" type="revolute">
+    <origin xyz="0 0 -0.02" rpy="1.5708 1.5708 0" />
+    <parent link="l_wrist_roll_link" />
+    <child link="l_wrist_pitch_link" />
+    <axis xyz="0 0 -1" />
+    <limit lower="-0.6981" upper="0.6981" effort="50000" velocity="500" />
+    <dynamics damping="0.7" friction="0.2"  />
+  </joint>
+  <link name="l_wrist_yaw_link">
+    <inertial>
+      <origin xyz="0.0096828 -0.0007914 2.2204E-16" rpy="0 0 0" />
+      <mass value="0.089949" />
+      <inertia
+        ixx="8E-04" ixy="-1E-04" ixz="0"
+        iyy="2E-04" iyz="0"
+        izz="2.2E-04" />
+    </inertial>
+    <visual>
+      <origin xyz="0 0 0" rpy="0 0 0" />
+      <geometry>
+        <mesh filename="package://upper_14/meshes/l_wrist_yaw_link.STL" />
+      </geometry>
+      <material name="">
+        <color rgba="0.68627 0.65882 0.63922 1" />
+      </material>
+    </visual>
+    <collision>
+      <origin xyz="0 0 0" rpy="0 0 0" />
+      <geometry>
+        <mesh filename="package://upper_14/meshes/l_wrist_yaw_link.STL" />
+      </geometry>
+    </collision>
+  </link>
+  <joint name="l_wrist_yaw" type="revolute">
+    <origin xyz="0.028 0 0" rpy="1.5708 -1.0276E-16 -6.9285E-31" />
+    <parent link="l_wrist_pitch_link" />
+    <child link="l_wrist_yaw_link" />
+    <axis xyz="0 0 1" />
+    <limit lower="-0.3141" upper="0.3141" effort="50000" velocity="500" />
+    <dynamics damping="0.7" friction="0.2"  />
+  </joint>
+  <link name="r_shoulder_roll_link">
+    <inertial>
+      <origin xyz="0.0033683 7.6367E-09 0.015946" rpy="0 0 0" />
+      <mass value="0.63417" />
+      <inertia
+        ixx="0.000315" ixy="0" ixz="5.2E-05"
+        iyy="0.000373" iyz="0"
+        izz="0.000525" />
+    </inertial>
+    <visual>
+      <origin xyz="0 0 0" rpy="0 0 0" />
+      <geometry>
+        <mesh filename="package://upper_14/meshes/r_shoulder_roll_link.STL" />
+      </geometry>
+      <material name="">
+        <color rgba="0.68627 0.65882 0.63922 1" />
+      </material>
+    </visual>
+    <collision>
+      <origin xyz="0 0 0" rpy="0 0 0" />
+      <geometry>
+        <mesh filename="package://upper_14/meshes/r_shoulder_roll_link.STL" />
+      </geometry>
+    </collision>
+  </link>
+  <joint name="r_shoulder_roll" type="continuous">
+    <origin xyz="-0.125 0 0.26" rpy="0 -1.5708 0" />
+    <parent link="upper_body_link" />
+    <child link="r_shoulder_roll_link" />
     <axis xyz="0 0 -1" />
     <limit effort="50000" velocity="500" />
-    <calibration rising="1" />
-    <dynamics damping="0.7" friction="0.1" />
-    <safety_controller k_velocity="1" />
-  </joint>
-  <link
-    name="l_wrist_pitch_link">
-    <inertial>
-      <origin
-        xyz="0.0009785 -2.8101E-08 -1.4985E-08"
-        rpy="0 0 0" />
-      <mass
-        value="0.13385" />
-      <inertia
-        ixx="2.1E-05"
-        ixy="0"
-        ixz="0"
-        iyy="2.2E-05"
-        iyz="0"
-        izz="2.2E-05" />
-    </inertial>
-    <visual>
-      <origin
-        xyz="0 0 0"
-        rpy="0 0 0" />
-      <geometry>
-        <mesh
-          filename="package://upper_14/meshes/l_wrist_pitch_link.STL" />
-      </geometry>
-      <material
-        name="">
-        <color
-          rgba="0.68627 0.65882 0.63922 1" />
-      </material>
-    </visual>
-    <collision>
-      <origin
-        xyz="0 0 0"
-        rpy="0 0 0" />
-      <geometry>
-        <mesh
-          filename="package://upper_14/meshes/l_wrist_pitch_link.STL" />
-      </geometry>
-    </collision>
-  </link>
-  <joint
-    name="l_wrist_pitch"
-    type="revolute">
-    <origin
-      xyz="0 0 -0.02"
-      rpy="1.5708 1.5708 0" />
-    <parent
-      link="l_wrist_roll_link" />
-    <child
-      link="l_wrist_pitch_link" />
-    <axis
-      xyz="0 0 -1" />
-    <limit
-      lower="-0.6981"
-      upper="0.6981"
-      effort="50000"
-      velocity="500" />
-    <calibration
-      rising="1" />
-    <dynamics
-      damping="0.7"
-      friction="0.1" />
-    <safety_controller
-      soft_upper="0.69"
-      soft_lower="-0.69"
-      k_position="1"
-      k_velocity="1" />
-  </joint>
-  <link
-    name="l_wrist_yaw_link">
-    <inertial>
-      <origin
-        xyz="0.0096828 -0.0007914 2.2204E-16"
-        rpy="0 0 0" />
-      <mass
-        value="0.089949" />
-      <inertia
-        ixx="8E-06"
-        ixy="-1E-06"
-        ixz="0"
-        iyy="2E-05"
-        iyz="0"
-        izz="2.2E-05" />
-    </inertial>
-    <visual>
-      <origin
-        xyz="0 0 0"
-        rpy="0 0 0" />
-      <geometry>
-        <mesh
-          filename="package://upper_14/meshes/l_wrist_yaw_link.STL" />
-      </geometry>
-      <material
-        name="">
-        <color
-          rgba="0.68627 0.65882 0.63922 1" />
-      </material>
-    </visual>
-    <collision>
-      <origin
-        xyz="0 0 0"
-        rpy="0 0 0" />
-      <geometry>
-        <mesh
-          filename="package://upper_14/meshes/l_wrist_yaw_link.STL" />
-      </geometry>
-    </collision>
-  </link>
-  <joint
-    name="l_wrist_yaw"
-    type="revolute">
-    <origin
-      xyz="0.028 0 0"
-      rpy="1.5708 -1.0276E-16 -6.9285E-31" />
-    <parent
-      link="l_wrist_pitch_link" />
-    <child
-      link="l_wrist_yaw_link" />
-    <axis
-      xyz="0 0 1" />
-    <limit
-      lower="-0.3141"
-      upper="0.3141"
-      effort="50000"
-      velocity="500" />
-    <calibration
-      rising="1" />
-    <dynamics
-      damping="0.7"
-      friction="0.1" />
-    <safety_controller
-      soft_upper="0.31"
-      soft_lower="-0.31"
-      k_position="1"
-      k_velocity="1" />
-  </joint>
-  <link
-    name="r_shoulder_roll_link">
-    <inertial>
-      <origin
-        xyz="0.0033683 7.6367E-09 0.015946"
-        rpy="0 0 0" />
-      <mass
-        value="0.63417" />
-      <inertia
-        ixx="0.000315"
-        ixy="0"
-        ixz="5.2E-05"
-        iyy="0.000373"
-        iyz="0"
-        izz="0.000525" />
-    </inertial>
-    <visual>
-      <origin
-        xyz="0 0 0"
-        rpy="0 0 0" />
-      <geometry>
-        <mesh
-          filename="package://upper_14/meshes/r_shoulder_roll_link.STL" />
-      </geometry>
-      <material
-        name="">
-        <color
-          rgba="0.68627 0.65882 0.63922 1" />
-      </material>
-    </visual>
-    <collision>
-      <origin
-        xyz="0 0 0"
-        rpy="0 0 0" />
-      <geometry>
-        <mesh
-          filename="package://upper_14/meshes/r_shoulder_roll_link.STL" />
-      </geometry>
-    </collision>
-  </link>
-  <joint
-    name="r_shoulder_roll"
-    type="continuous">
-    <origin
-      xyz="-0.125 0 0.26"
-      rpy="0 -1.5708 0" />
-    <parent
-      link="upper_body_link" />
-    <child
-      link="r_shoulder_roll_link" />
-    <axis
-      xyz="0 0 -1" />
-    <limit
-      effort="50000"
-      velocity="500" />
-    <calibration
-      rising="1" />
-    <dynamics
-      damping="0.7"
-      friction="0.1" />
-    <safety_controller
-      k_velocity="1" />
-  </joint>
-  <link
-    name="r_shoulder_pitch_link">
-    <inertial>
-      <origin
-        xyz="0.0032993 -5.9585E-10 0.00098089"
-        rpy="0 0 0" />
-      <mass
-        value="1.0724" />
-      <inertia
-        ixx="0.000841"
-        ixy="0"
-        ixz="5.4E-05"
-        iyy="0.000973"
-        iyz="0"
+    <dynamics damping="0.7" friction="0.2"  />
+  </joint>
+  <link name="r_shoulder_pitch_link">
+    <inertial>
+      <origin xyz="0.0032993 -5.9585E-10 0.00098089" rpy="0 0 0" />
+      <mass value="1.0724" />
+      <inertia
+        ixx="0.000841" ixy="0" ixz="5.4E-05"
+        iyy="0.000973" iyz="0"
         izz="0.000606" />
     </inertial>
     <visual>
-      <origin
-        xyz="0 0 0"
-        rpy="0 0 0" />
-      <geometry>
-        <mesh
-          filename="package://upper_14/meshes/r_shoulder_pitch_link.STL" />
-      </geometry>
-      <material
-        name="">
-        <color
-          rgba="0.68627 0.65882 0.63922 1" />
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