Commit message: Robot Ready
The robot is current ready for the simulation. There's an issue that due to the lacking of  controller, the model will collapse to origin unless the inertia matrix is increased to above e-4 level.

File: robots/src/upper_14/urdf/lita.xacro (robot description, xacro)
@@ -1,3 +1,2 @@
-<?xml version="1.0"?>
 <robot name="upper_14" xmlns:xacro="http://www.ros.org/wiki/xacro">
   <!--fix the upper_body_link-->
@@ -37,5 +36,5 @@
     <parent link="upper_body_link" />
     <child link="l_shoulder_roll_link" />
-    <axis xyz="0 0 -1" />
+    <axis xyz="0 0 1" />
     <dynamics damping="0.7" />
   </joint>
@@ -96,7 +95,5 @@
     <axis xyz="0 0 -1" />
     <limit lower="-0.6981" upper="1.7104" effort="50000" velocity="500" />
-    <calibration rising="1" />
-    <dynamics damping="0.7" friction="0.1" />
-    <safety_controller soft_upper="1.7" soft_lower="-0.69" k_position="1" k_velocity="1" />
+    <dynamics damping="0.7"   />
   </joint>
   <link name="l_shoulder_yaw_link">
@@ -131,7 +128,5 @@
     <axis xyz="0 0 1" />
     <limit lower="-0.1396" upper="1.6231" effort="50000" velocity="500" />
-    <calibration rising="1" />
-    <dynamics damping="0.7" friction="0.1" />
-    <safety_controller soft_upper="1.61" soft_lower="-0.13" k_position="1" k_velocity="1" />
+    <dynamics damping="0.7"   />
   </joint>
   <link name="l_elbow_link">
@@ -149,6 +144,5 @@
         <mesh filename="package://upper_14/meshes/l_elbow_link.STL" />
       </geometry>
-      <material
-        name="">
+      <material name="">
         <color rgba="0.68627 0.65882 0.63922 1" />
       </material>
@@ -167,7 +161,5 @@
     <axis xyz="0 0 1" />
     <limit lower="-0.7853" upper="2.4085" effort="50000" velocity="500" />
-    <calibration rising="1" />
-    <dynamics damping="0.7" friction="0.1" />
-    <safety_controller soft_upper="2.4" soft_lower="-0.78" k_position="1" k_velocity="1" />
+    <dynamics damping="0.7"   />
   </joint>
   <link name="l_wrist_roll_link">
@@ -185,6 +177,5 @@
         <mesh filename="package://upper_14/meshes/l_wrist_roll_link.STL" />
       </geometry>
-      <material
-        name="">
+      <material name="">
         <color rgba="0.68627 0.65882 0.63922 1" />
       </material>
@@ -201,610 +192,304 @@
     <parent link="l_elbow_link" />
     <child link="l_wrist_roll_link" />
-    <axis xyz="0 0 -1" />
+    <axis xyz="0 0 1" />
     <limit effort="50000" velocity="500" />
-    <calibration rising="1" />
-    <dynamics damping="0.7" friction="0.1" />
-    <safety_controller k_velocity="1" />
-  </joint>
-  <link
-    name="l_wrist_pitch_link">
-    <inertial>
-      <origin
-        xyz="0.0009785 -2.8101E-08 -1.4985E-08"
-        rpy="0 0 0" />
-      <mass
-        value="0.13385" />
-      <inertia
-        ixx="2.1E-05"
-        ixy="0"
-        ixz="0"
-        iyy="2.2E-05"
-        iyz="0"
+    <dynamics damping="0.7"   />
+  </joint>
+  <link name="l_wrist_pitch_link">
+    <inertial>
+      <origin xyz="0.0009785 -2.8101E-08 -1.4985E-08" rpy="0 0 0" />
+      <mass value="0.13385" />
+      <inertia
+        ixx="2.1E-05" ixy="0" ixz="0"
+        iyy="2.2E-05" iyz="0"
         izz="2.2E-05" />
     </inertial>
     <visual>
-      <origin
-        xyz="0 0 0"
-        rpy="0 0 0" />
-      <geometry>
-        <mesh
-          filename="package://upper_14/meshes/l_wrist_pitch_link.STL" />
-      </geometry>
-      <material
-        name="">
-        <color
-          rgba="0.68627 0.65882 0.63922 1" />
-      </material>
-    </visual>
-    <collision>
-      <origin
-        xyz="0 0 0"
-        rpy="0 0 0" />
-      <geometry>
-        <mesh
-          filename="package://upper_14/meshes/l_wrist_pitch_link.STL" />
-      </geometry>
-    </collision>
-  </link>
-  <joint
-    name="l_wrist_pitch"
-    type="revolute">
-    <origin
-      xyz="0 0 -0.02"
-      rpy="1.5708 1.5708 0" />
-    <parent
-      link="l_wrist_roll_link" />
-    <child
-      link="l_wrist_pitch_link" />
-    <axis
-      xyz="0 0 -1" />
-    <limit
-      lower="-0.6981"
-      upper="0.6981"
-      effort="50000"
-      velocity="500" />
-    <calibration
-      rising="1" />
-    <dynamics
-      damping="0.7"
-      friction="0.1" />
-    <safety_controller
-      soft_upper="0.69"
-      soft_lower="-0.69"
-      k_position="1"
-      k_velocity="1" />
-  </joint>
-  <link
-    name="l_wrist_yaw_link">
-    <inertial>
-      <origin
-        xyz="0.0096828 -0.0007914 2.2204E-16"
-        rpy="0 0 0" />
-      <mass
-        value="0.089949" />
-      <inertia
-        ixx="8E-06"
-        ixy="-1E-06"
-        ixz="0"
-        iyy="2E-05"
-        iyz="0"
+      <origin xyz="0 0 0" rpy="0 0 0" />
+      <geometry>
+        <mesh filename="package://upper_14/meshes/l_wrist_pitch_link.STL" />
+      </geometry>
+      <material name="">
+        <color rgba="0.68627 0.65882 0.63922 1" />
+      </material>
+    </visual>
+    <collision>
+      <origin xyz="0 0 0" rpy="0 0 0" />
+      <geometry>
+        <mesh filename="package://upper_14/meshes/l_wrist_pitch_link.STL" />
+      </geometry>
+    </collision>
+  </link>
+  <joint name="l_wrist_pitch" type="revolute">
+    <origin xyz="0 0 -0.02" rpy="1.5708 1.5708 0" />
+    <parent link="l_wrist_roll_link" />
+    <child link="l_wrist_pitch_link" />
+    <axis xyz="0 0 -1" />
+    <limit lower="-0.6981" upper="0.6981" effort="50000" velocity="500" />
+    <dynamics damping="0.7"   />
+  </joint>
+  <link name="l_wrist_yaw_link">
+    <inertial>
+      <origin xyz="0.0096828 -0.0007914 2.2204E-16" rpy="0 0 0" />
+      <mass value="0.089949" />
+      <inertia
+        ixx="8E-06" ixy="-1E-06" ixz="0"
+        iyy="2E-05" iyz="0"
         izz="2.2E-05" />
     </inertial>
     <visual>
-      <origin
-        xyz="0 0 0"
-        rpy="0 0 0" />
-      <geometry>
-        <mesh
-          filename="package://upper_14/meshes/l_wrist_yaw_link.STL" />
-      </geometry>
-      <material
-        name="">
-        <color
-          rgba="0.68627 0.65882 0.63922 1" />
-      </material>
-    </visual>
-    <collision>
-      <origin
-        xyz="0 0 0"
-        rpy="0 0 0" />
-      <geometry>
-        <mesh
-          filename="package://upper_14/meshes/l_wrist_yaw_link.STL" />
-      </geometry>
-    </collision>
-  </link>
-  <joint
-    name="l_wrist_yaw"
-    type="revolute">
-    <origin
-      xyz="0.028 0 0"
-      rpy="1.5708 -1.0276E-16 -6.9285E-31" />
-    <parent
-      link="l_wrist_pitch_link" />
-    <child
-      link="l_wrist_yaw_link" />
-    <axis
-      xyz="0 0 1" />
-    <limit
-      lower="-0.3141"
-      upper="0.3141"
-      effort="50000"
-      velocity="500" />
-    <calibration
-      rising="1" />
-    <dynamics
-      damping="0.7"
-      friction="0.1" />
-    <safety_controller
-      soft_upper="0.31"
-      soft_lower="-0.31"
-      k_position="1"
-      k_velocity="1" />
-  </joint>
-  <link
-    name="r_shoulder_roll_link">
-    <inertial>
-      <origin
-        xyz="0.0033683 7.6367E-09 0.015946"
-        rpy="0 0 0" />
-      <mass
-        value="0.63417" />
-      <inertia
-        ixx="0.000315"
-        ixy="0"
-        ixz="5.2E-05"
-        iyy="0.000373"
-        iyz="0"
+      <origin xyz="0 0 0" rpy="0 0 0" />
+      <geometry>
+        <mesh filename="package://upper_14/meshes/l_wrist_yaw_link.STL" />
+      </geometry>
+      <material name="">
+        <color rgba="0.68627 0.65882 0.63922 1" />
+      </material>
+    </visual>
+    <collision>
+      <origin xyz="0 0 0" rpy="0 0 0" />
+      <geometry>
+        <mesh filename="package://upper_14/meshes/l_wrist_yaw_link.STL" />
+      </geometry>
+    </collision>
+  </link>
+  <joint name="l_wrist_yaw" type="revolute">
+    <origin xyz="0.028 0 0" rpy="1.5708 -1.0276E-16 -6.9285E-31" />
+    <parent link="l_wrist_pitch_link" />
+    <child link="l_wrist_yaw_link" />
+    <axis xyz="0 0 1" />
+    <limit lower="-0.3141" upper="0.3141" effort="50000" velocity="500" />
+    <dynamics damping="0.7"   />
+  </joint>
+  <link name="r_shoulder_roll_link">
+    <inertial>
+      <origin xyz="0.0033683 7.6367E-09 0.015946" rpy="0 0 0" />
+      <mass value="0.63417" />
+      <inertia
+        ixx="0.000315" ixy="0" ixz="5.2E-05"
+        iyy="0.000373" iyz="0"
         izz="0.000525" />
     </inertial>
     <visual>
-      <origin
-        xyz="0 0 0"
-        rpy="0 0 0" />
-      <geometry>
-        <mesh
-          filename="package://upper_14/meshes/r_shoulder_roll_link.STL" />
-      </geometry>
-      <material
-        name="">
-        <color
-          rgba="0.68627 0.65882 0.63922 1" />
-      </material>
-    </visual>
-    <collision>
-      <origin
-        xyz="0 0 0"
-        rpy="0 0 0" />
-      <geometry>
-        <mesh
-          filename="package://upper_14/meshes/r_shoulder_roll_link.STL" />
-      </geometry>
-    </collision>
-  </link>
-  <joint
-    name="r_shoulder_roll"
-    type="continuous">
-    <origin
-      xyz="-0.125 0 0.26"
-      rpy="0 -1.5708 0" />
-    <parent
-      link="upper_body_link" />
-    <child
-      link="r_shoulder_roll_link" />
-    <axis
-      xyz="0 0 -1" />
-    <limit
-      effort="50000"
-      velocity="500" />
-    <calibration
-      rising="1" />
-    <dynamics
-      damping="0.7"
-      friction="0.1" />
-    <safety_controller
-      k_velocity="1" />
-  </joint>
-  <link
-    name="r_shoulder_pitch_link">
-    <inertial>
-      <origin
-        xyz="0.0032993 -5.9585E-10 0.00098089"
-        rpy="0 0 0" />
-      <mass
-        value="1.0724" />
-      <inertia
-        ixx="0.000841"
-        ixy="0"
-        ixz="5.4E-05"
-        iyy="0.000973"
-        iyz="0"
+      <origin xyz="0 0 0" rpy="0 0 0" />
+      <geometry>
+        <mesh filename="package://upper_14/meshes/r_shoulder_roll_link.STL" />
+      </geometry>
+      <material name="">
+        <color rgba="0.68627 0.65882 0.63922 1" />
+      </material>
+    </visual>
+    <collision>
+      <origin xyz="0 0 0" rpy="0 0 0" />
+      <geometry>
+        <mesh filename="package://upper_14/meshes/r_shoulder_roll_link.STL" />
+      </geometry>
+    </collision>
+  </link>
+  <joint name="r_shoulder_roll" type="continuous">
+    <origin xyz="-0.125 0 0.26" rpy="0 -1.5708 0" />
+    <parent link="upper_body_link" />
+    <child link="r_shoulder_roll_link" />
+    <axis xyz="0 0 -1" />
+    <limit effort="50000" velocity="500" />
+    <dynamics damping="0.7"   />
+  </joint>
+  <link name="r_shoulder_pitch_link">
+    <inertial>
+      <origin xyz="0.0032993 -5.9585E-10 0.00098089" rpy="0 0 0" />
+      <mass value="1.0724" />
+      <inertia
+        ixx="0.000841" ixy="0" ixz="5.4E-05"
+        iyy="0.000973" iyz="0"
         izz="0.000606" />
     </inertial>
     <visual>
-      <origin
-        xyz="0 0 0"
-        rpy="0 0 0" />
-      <geometry>
-        <mesh
-          filename="package://upper_14/meshes/r_shoulder_pitch_link.STL" />
-      </geometry>
-      <material
-        name="">
-        <color
-          rgba="0.68627 0.65882 0.63922 1" />
-      </material>
-    </visual>
-    <collision>
-      <origin
-        xyz="0 0 0"
-        rpy="0 0 0" />
-      <geometry>
-        <mesh
-          filename="package://upper_14/meshes/r_shoulder_pitch_link.STL" />
-      </geometry>
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
Commit message: Revert robot ready

File: robots/src/upper_14/urdf/lita.xacro (robot description, xacro)
@@ -36,4 +36,5 @@
     <parent link="upper_body_link" />
     <child link="l_shoulder_roll_link" />
+    <axis xyz="0 0 1" />
     <dynamics damping="0.7" friction="0.2"/>
   </joint>
@@ -94,7 +95,5 @@
     <axis xyz="0 0 -1" />
     <limit lower="-0.6981" upper="1.7104" effort="50000" velocity="500" />
-    <calibration rising="1" />
-    <dynamics damping="0.7" friction="0.1" />
-    <safety_controller soft_upper="1.7" soft_lower="-0.69" k_position="1" k_velocity="1" />
+    <dynamics damping="0.7" friction="0.2"  />
   </joint>
   <link name="l_shoulder_yaw_link">
@@ -129,7 +128,5 @@
     <axis xyz="0 0 1" />
     <limit lower="-0.1396" upper="1.6231" effort="50000" velocity="500" />
-    <calibration rising="1" />
-    <dynamics damping="0.7" friction="0.1" />
-    <safety_controller soft_upper="1.61" soft_lower="-0.13" k_position="1" k_velocity="1" />
+    <dynamics damping="0.7" friction="0.2"  />
   </joint>
   <link name="l_elbow_link">
@@ -164,7 +161,5 @@
     <axis xyz="0 0 1" />
     <limit lower="-0.7853" upper="2.4085" effort="50000" velocity="500" />
-    <calibration rising="1" />
-    <dynamics damping="0.7" friction="0.1" />
-    <safety_controller soft_upper="2.4" soft_lower="-0.78" k_position="1" k_velocity="1" />
+    <dynamics damping="0.7" friction="0.2"  />
   </joint>
   <link name="l_wrist_roll_link">
@@ -199,7 +194,5 @@
     <axis xyz="0 0 1" />
     <limit effort="50000" velocity="500" />
-    <calibration rising="1" />
-    <dynamics damping="0.7" friction="0.1" />
-    <safety_controller k_velocity="1" />
+    <dynamics damping="0.7" friction="0.2"  />
   </joint>
   <link name="l_wrist_pitch_link">
@@ -208,10 +201,7 @@
       <mass value="0.13385" />
       <inertia
-        ixx="2.1E-05"
-        ixy="0"
-        ixz="0"
-        iyy="2.2E-05"
-        iyz="0"
-        izz="2.2E-05" />
+        ixx="2.1E-03" ixy="0" ixz="0"
+        iyy="2.2E-03" iyz="0"
+        izz="2.2E-03" />
     </inertial>
     <visual>
@@ -231,31 +221,11 @@
     </collision>
   </link>
-  <joint
-    name="l_wrist_pitch"
-    type="revolute">
-    <origin
-      xyz="0 0 -0.02"
-      rpy="1.5708 1.5708 0" />
-    <parent
-      link="l_wrist_roll_link" />
-    <child
-      link="l_wrist_pitch_link" />
-    <axis
-      xyz="0 0 -1" />
-    <limit
-      lower="-0.6981"
-      upper="0.6981"
-      effort="50000"
-      velocity="500" />
-    <calibration
-      rising="1" />
-    <dynamics
-      damping="0.7"
-      friction="0.1" />
-    <safety_controller
-      soft_upper="0.69"
-      soft_lower="-0.69"
-      k_position="1"
-      k_velocity="1" />
+  <joint name="l_wrist_pitch" type="revolute">
+    <origin xyz="0 0 -0.02" rpy="1.5708 1.5708 0" />
+    <parent link="l_wrist_roll_link" />
+    <child link="l_wrist_pitch_link" />
+    <axis xyz="0 0 -1" />
+    <limit lower="-0.6981" upper="0.6981" effort="50000" velocity="500" />
+    <dynamics damping="0.7" friction="0.2"  />
   </joint>
   <link name="l_wrist_yaw_link">
@@ -264,10 +234,7 @@
       <mass value="0.089949" />
       <inertia
-        ixx="8E-06"
-        ixy="-1E-06"
-        ixz="0"
-        iyy="2E-05"
-        iyz="0"
-        izz="2.2E-05" />
+        ixx="8E-04" ixy="-1E-04" ixz="0"
+        iyy="2E-04" iyz="0"
+        izz="2.2E-04" />
     </inertial>
     <visual>
@@ -287,31 +254,11 @@
     </collision>
   </link>
-  <joint
-    name="l_wrist_yaw"
-    type="revolute">
-    <origin
-      xyz="0.028 0 0"
-      rpy="1.5708 -1.0276E-16 -6.9285E-31" />
-    <parent
-      link="l_wrist_pitch_link" />
-    <child
-      link="l_wrist_yaw_link" />
-    <axis
-      xyz="0 0 1" />
-    <limit
-      lower="-0.3141"
-      upper="0.3141"
-      effort="50000"
-      velocity="500" />
-    <calibration
-      rising="1" />
-    <dynamics
-      damping="0.7"
-      friction="0.1" />
-    <safety_controller
-      soft_upper="0.31"
-      soft_lower="-0.31"
-      k_position="1"
-      k_velocity="1" />
+  <joint name="l_wrist_yaw" type="revolute">
+    <origin xyz="0.028 0 0" rpy="1.5708 -1.0276E-16 -6.9285E-31" />
+    <parent link="l_wrist_pitch_link" />
+    <child link="l_wrist_yaw_link" />
+    <axis xyz="0 0 1" />
+    <limit lower="-0.3141" upper="0.3141" effort="50000" velocity="500" />
+    <dynamics damping="0.7" friction="0.2"  />
   </joint>
   <link name="r_shoulder_roll_link">
@@ -340,26 +287,11 @@
     </collision>
   </link>
-  <joint
-    name="r_shoulder_roll"
-    type="continuous">
-    <origin
-      xyz="-0.125 0 0.26"
-      rpy="0 -1.5708 0" />
-    <parent
-      link="upper_body_link" />
-    <child
-      link="r_shoulder_roll_link" />
-    <axis
-      xyz="0 0 -1" />
-    <limit
-      effort="50000"
-      velocity="500" />
-    <calibration
-      rising="1" />
-    <dynamics
-      damping="0.7"
-      friction="0.1" />
-    <safety_controller
-      k_velocity="1" />
+  <joint name="r_shoulder_roll" type="continuous">
+    <origin xyz="-0.125 0 0.26" rpy="0 -1.5708 0" />
+    <parent link="upper_body_link" />
+    <child link="r_shoulder_roll_link" />
+    <axis xyz="0 0 -1" />
+    <limit effort="50000" velocity="500" />
+    <dynamics damping="0.7" friction="0.2"  />
   </joint>
   <link name="r_shoulder_pitch_link">
@@ -388,31 +320,11 @@
     </collision>
   </link>
-  <joint
-    name="r_shoulder_pitch"
-    type="revolute">
-    <origin
-      xyz="-0.0037133 0 0.052049"
-      rpy="-1.5708 -1.5708 0" />
-    <parent
-      link="r_shoulder_roll_link" />
-    <child
-      link="r_shoulder_pitch_link" />
-    <axis
-      xyz="0 0 -1" />
-    <limit
-      lower="-0.6981"
-      upper="1.7104"
-      effort="50000"
-      velocity="500" />
-    <calibration
-      rising="1" />
-    <dynamics
-      damping="0.7"
-      friction="0.1" />
-    <safety_controller
-      soft_upper="1.7"
-      soft_lower="-0.69"
-      k_position="1"
-      k_velocity="1" />
+  <joint name="r_shoulder_pitch" type="revolute">
+    <origin xyz="-0.0037133 0 0.052049" rpy="-1.5708 -1.5708 0" />
+    <parent link="r_shoulder_roll_link" />
+    <child link="r_shoulder_pitch_link" />
+    <axis xyz="0 0 -1" />
+    <limit lower="-0.6981" upper="1.7104" effort="50000" velocity="500" />
+    <dynamics damping="0.7" friction="0.2"  />
   </joint>
   <link name="r_shoulder_yaw_link">
@@ -441,30 +353,11 @@
     </collision>
   </link>
-  <joint
-    name="r_shoulder_yaw"
-    type="revolute">
-    <origin
-      xyz="0.055 0 0"
-      rpy="-1.5708 3.2819E-17 -4.3368E-18" />
-    <parent
-      link="r_shoulder_pitch_link" />
-    <child
-      link="r_shoulder_yaw_link" />
-    <axis
-      xyz="0 0 1" />
-    <limit
-      lower="-0.1396"
-      upper="1.6231"
-      effort="50000"
-      velocity="500" />
-    <calibration
-      rising="1" />
-    <dynamics
-      damping="0.7"
-      friction="0.1" />
-    <safety_controller
-      soft_upper="1.61"
-      soft_lower="-0.13"
-      k_velocity="0" />
+  <joint name="r_shoulder_yaw" type="revolute">
+    <origin xyz="0.055 0 0" rpy="-1.5708 3.2819E-17 -4.3368E-18" />
+    <parent link="r_shoulder_pitch_link" />
+    <child link="r_shoulder_yaw_link" />
+    <axis xyz="0 0 1" />
+    <limit lower="-0.1396" upper="1.6231" effort="50000" velocity="500" />
+    <dynamics damping="0.7" friction="0.2"  />
   </joint>
   <link name="r_elbow_link">
@@ -493,31 +386,11 @@
     </collision>
   </link>
-  <joint
-    name="r_elbow"
-    type="revolute">
-    <origin
-      xyz="0.1903 0 0"
-      rpy="1.2818E-16 -4.3368E-18 -2.8339E-19" />
-    <parent
-      link="r_shoulder_yaw_link" />
-    <child
-      link="r_elbow_link" />
-    <axis
-      xyz="0 0 1" />
-    <limit
-      lower="-0.7853"
-      upper="2.4085"
-      effort="50000"
-      velocity="500" />
-    <calibration
-      rising="1" />
-    <dynamics
-      damping="0.7"
-      friction="0.1" />
-    <safety_controller
-      soft_upper="2.4"
-      soft_lower="-0.78"
-      k_position="1"
-      k_velocity="1" />
+  <joint name="r_elbow" type="revolute">
+    <origin xyz="0.1903 0 0" rpy="1.2818E-16 -4.3368E-18 -2.8339E-19" />
+    <parent link="r_shoulder_yaw_link" />
+    <child link="r_elbow_link" />
+    <axis xyz="0 0 1" />
+    <limit lower="-0.7853" upper="2.4085" effort="50000" velocity="500" />
+    <dynamics damping="0.7" friction="0.2"  />
   </joint>
   <link name="r_wrist_roll_link">
@@ -526,10 +399,7 @@
       <mass value="0.033212" />
       <inertia
-        ixx="3E-06"
-        ixy="0"
-        ixz="0"
-        iyy="6E-06"
-        iyz="0"
-        izz="8E-06" />
+        ixx="3E-04" ixy="0" ixz="0"
+        iyy="6E-04" iyz="0"
+        izz="8E-04" />
     </inertial>
     <visual>
@@ -549,26 +419,11 @@
     </collision>
   </link>
-  <joint
-    name="r_wrist_roll"
-    type="continuous">
-    <origin
-      xyz="0.21 0 0"
-      rpy="0 1.5708 0" />
-    <parent
-      link="r_elbow_link" />
-    <child
-      link="r_wrist_roll_link" />
-    <axis
-      xyz="0 0 -1" />
-    <limit
-      effort="50000"
-      velocity="500" />
-    <calibration
-      rising="1" />
-    <dynamics
-      damping="0.7"
-      friction="0.1" />
-    <safety_controller
-      k_velocity="1" />
+  <joint name="r_wrist_roll" type="continuous">
+    <origin xyz="0.21 0 0" rpy="0 1.5708 0" />
+    <parent link="r_elbow_link" />
+    <child link="r_wrist_roll_link" />
+    <axis xyz="0 0 -1" />
+    <limit effort="50000" velocity="500" />
+    <dynamics damping="0.7" friction="0.2"  />
   </joint>
   <link name="r_wrist_pitch_link">
@@ -577,10 +432,7 @@
       <mass value="0.13385" />
       <inertia
-        ixx="2.1E-05"
-        ixy="0"
-        ixz="0"
-        iyy="2.2E-05"
-        iyz="0"
-        izz="2.2E-05" />
+        ixx="2.1E-04" ixy="0" ixz="0"
+        iyy="2.2E-04" iyz="0"
+        izz="2.2E-04" />
     </inertial>
     <visual>
@@ -600,31 +452,11 @@
     </collision>
   </link>
-  <joint
-    name="r_wrist_pitch"
-    type="revolute">
-    <origin
-      xyz="0 0 0.02"
-      rpy="1.5708 -1.5708 0" />
-    <parent
-      link="r_wrist_roll_link" />
-    <child
-      link="r_wrist_pitch_link" />
-    <axis
-      xyz="0 0 -1" />
-    <limit
-      lower="-0.6981"
-      upper="0.6981"
-      effort="50000"
-      velocity="500" />
-    <calibration
-      rising="1" />
-    <dynamics
-      damping="0.7"
-      friction="0.1" />
-    <safety_controller
-      soft_upper="0.69"
-      soft_lower="-0.69"
-      k_position="1"
-      k_velocity="1" />
+  <joint name="r_wrist_pitch" type="revolute">
+    <origin xyz="0 0 0.02" rpy="1.5708 -1.5708 0" />
+    <parent link="r_wrist_roll_link" />
+    <child link="r_wrist_pitch_link" />
+    <axis xyz="0 0 -1" />
+    <limit lower="-0.6981" upper="0.6981" effort="50000" velocity="500" />
+    <dynamics damping="0.7" friction="0.2"  />
   </joint>
   <link name="r_wrist_yaw_link">
@@ -633,10 +465,7 @@
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